File: Fichiers KiCad/Kicad Projet Capteur.kicad_pcb (KiCad board)
At the start: 2 copper layers, 68.6 x 53.3 mm, 24 parts, among them J1 Power, J2 Digital/PWM, J3 Analog, J4 Digital/PWM, U1 LTC1050#CN8, U2 MCP41050

Commit message: Amélioration layout KiCad
OLED +
Connections:
- J2 pad 6: /12 -> PWM/SS
- J2 pad 8: PWM/SS -> /*10
- SSD1306 pad 3: 5V -> GND
- SSD1306 pad 4: GND -> 5V
Routing:
- net GND: track 8.83 -> 0.18 mm
- net MOSI: track 30.2 -> 24.8 mm
- net 5V: track 169.8 -> 172.9 mm
- net PWM/SS: track 7.60 -> 9.70 mm
- net RXD: track 9.17 -> 10.4 mm
- net A: track 37.4 -> 38.4 mm
- added copper zone on B.Cu, net GND
- removed copper zone on F.Cu, net GND

Commit message: Nouveau PCB + Nouveau GIF
Plan de masse un peu plus propre et mise à jour du GIF
Routing:
- net MOSI: track 24.8 -> 24.3 mm
Changed lines of the file:
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@@
     (pad_to_mask_clearance 0)
     (aux_axis_origin 100 100)
-    (grid_origin 100 100)
     (pcbplotparams
       (layerselection 0x0000030_80000001)
@@
     (pad "1" thru_hole rect (at 0 0 180) (size 2 2) (drill 1) (layers "*.Cu" "*.Mask")
       (net 12 "5V") (pinfunction "5V") (pintype "passive"))
-    (pad "2" thru_hole oval (at 0 2.54 180) (size 2 2) (drill 1) (layers "*.Cu" "*.Mask")
+    (pad "2" thru_hole circle (at 0 2.54 180) (size 2 2) (drill 1) (layers "*.Cu" "*.Mask")
       (net 22 "Net-(Capteur-Graphite1-Ampli)") (pinfunction "Ampli") (pintype "passive"))
     (model "${KICAD6_3DMODEL_DIR}/Connector_PinSocket_2.54mm.3dshapes/PinSocket_1x02_P2.54mm_Vertical.wrl"
@@
     (property "Sheetname" "")
     (attr through_hole)
-    (fp_text reference "Pot1" (at 0 -2.77) (layer "F.SilkS")
+    (fp_text reference "Pot1" (at 2.515 5.08 90) (layer "F.SilkS")
         (effects (font (size 1 1) (thickness 0.15)))
     )
@@
     (property "ki_keywords" "R res resistor")
     (attr through_hole)
-    (fp_text reference "R1" (at 2.54 0 90) (layer "F.SilkS")
+    (fp_text reference "R1" (at 2.54 0 -180) (layer "F.SilkS")
         (effects (font (size 1 1) (thickness 0.15)))
     )
@@
     (fp_line (start 5.08 0) (end 4.34 0)
       (stroke (width 0.1) (type solid)) (layer "F.Fab"))
-    (pad "1" thru_hole circle (at 0 0 270) (size 2 2) (drill 0.8) (layers "*.Cu" "*.Mask" "F.Adhes")
+    (pad "1" thru_hole circle (at 0 0 270) (size 2 2) (drill 0.8) (layers "*.Cu" "*.Mask")
       (net 5 "Net-(U1-+IN)") (pintype "passive"))
     (pad "2" thru_hole circle (at 5.08 0 270) (size 2 2) (drill 0.8) (layers "*.Cu" "*.Mask" "B.SilkS")
@@
     (property "ki_keywords" "cap capacitor")
     (attr through_hole)
-    (fp_text reference "C4" (at 2.5 0 90) (layer "F.SilkS")
+    (fp_text reference "C4" (at 2.5 0 180) (layer "F.SilkS")
         (effects (font (size 1 1) (thickness 0.15)))
     )
@@
   (segment (start 128.956 49.2) (end 128.956 51.361) (width 0.5) (layer "B.Cu") (net 13))
   (segment (start 128.956 51.361) (end 134.29 56.695) (width 0.5) (layer "B.Cu") (net 13))
-  (segment (start 139.125 60.075) (end 140.4 58.8) (width 0.5) (layer "B.Cu") (net 20))
-  (segment (start 135.025 60.075) (end 139.125 60.075) (width 0.5) (layer "B.Cu") (net 20))
+  (segment (start 131.75 56.695) (end 131.75 56.8) (width 0.5) (layer "B.Cu") (net 20))
+  (segment (start 134.036 50.43) (end 134.036 49.2) (width 0.5) (layer "B.Cu") (net 20))
+  (segment (start 137.356 53.75) (end 134.036 50.43) (width 0.5) (layer "B.Cu") (net 20))
+  (segment (start 140.4 54.875) (end 139.275 53.75) (width 0.5) (layer "B.Cu") (net 20))
+  (segment (start 131.75 56.8) (end 134.31 59.36) (width 0.5) (layer "B.Cu") (net 20))
+  (segment (start 134.29 49.454) (end 134.036 49.2) (width 0.5) (layer "B.Cu") (net 20))
   (segment (start 140.4 58.8) (end 140.4 54.875) (width 0.5) (layer "B.Cu") (net 20))
-  (segment (start 131.75 56.8) (end 135.025 60.075) (width 0.5) (layer "B.Cu") (net 20))
-  (segment (start 140.4 54.875) (end 139.275 53.75) (width 0.5) (layer "B.Cu") (net 20))
-  (segment (start 134.29 49.454) (end 134.036 49.2) (width 0.5) (layer "B.Cu") (net 20))
+  (segment (start 139.84 59.36) (end 140.4 58.8) (width 0.5) (layer "B.Cu") (net 20))
+  (segment (start 131.75 56.695) (end 131.75 56.82) (width 0.5) (layer "B.Cu") (net 20))
+  (segment (start 134.31 59.36) (end 139.84 59.36) (width 0.5) (layer "B.Cu") (net 20))
   (segment (start 139.275 53.75) (end 137.356 53.75) (width 0.5) (layer "B.Cu") (net 20))
-  (segment (start 137.356 53.75) (end 134.036 50.43) (width 0.5) (layer "B.Cu") (net 20))
-  (segment (start 131.75 56.695) (end 131.75 56.82) (width 0.5) (layer "B.Cu") (net 20))
-  (segment (start 134.036 50.43) (end 134.036 49.2) (width 0.5) (layer "B.Cu") (net 20))
   (segment (start 131.75 56.82) (end 131.496 56.566) (width 0.5) (layer "B.Cu") (net 20))
-  (segment (start 131.75 56.695) (end 131.75 56.8) (width 0.5) (layer "B.Cu") (net 20))
   (segment (start 131.496 51.361) (end 131.496 49.2) (width 0.5) (layer "B.Cu") (net 21))
   (segment (start 136.83 56.695) (end 131.496 51.361) (width 0.5) (layer "B.Cu") (net 21))
@@
     (polygon
       (pts
-        (xy 100 46.66)
-        (xy 168.58 46.66)
-        (xy 168.58 100)
-        (xy 100 100)
+        (xy 115.24 46.66)
+        (xy 115.24 53.01)
+        (xy 125.4 53.01)
+        (xy 125.4 59.36)
+        (xy 113.97 59.36)
+        (xy 108.89 64.44)
+        (xy 108.89 70.79)
+        (xy 112.7 74.6)
+        (xy 112.7 73.33)
+        (xy 112.7 91.11)
+        (xy 116.51 94.92)
+        (xy 116.51 100)
+        (xy 166.04 100)
+        (xy 166.04 96.19)
+        (xy 166.04 94.92)
+        (xy 166.04 79.68)
+        (xy 159.69 73.33)
+        (xy 159.69 72.06)
+        (xy 163.5 68.25)
+        (xy 163.5 61.9)
+        (xy 162.23 60.63)
+        (xy 162.23 53.01)
+        (xy 162.23 53.01)
+        (xy 166.04 53.01)
+        (xy 166.04 49.2)
+        (xy 163.5 46.66)
+        (xy 116.51 46.66)
       )
     )
